File: main_pcb/kicad_6/CV_generators.kicad_sch (KiCad schematic)
At the start: 6 parts

Commit message: Update rev 0.1, fix VCA tails, add local 2v5 regs, change some pot footprints
Parts:
- removed RV603: 100k, custom_footprints:Alpha_RD901F, symbol Device:R_Potentiometer
Connections:
- net VCA_env/OUT is gone; now on net VCA_CV: TP601.1
Other:
- added sheet gate_conditioner (gate_conditioner.kicad_sch)
- sheet VCA_env ports: added ~{TRIG}; removed none
- sheet VCF_env ports: added ~{TRIG}; removed none
- note removed: "master volume"
- moved on the sheet: RV601, RV602, TP601, TP602, TP603

Commit message: Add mod-wheel VCA, fix occasional VCO freq locking
Other:
- sheet LFO ports: added DEPTH_CV_IN; removed none
Changed lines of the file:
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@@
   (title_block
     (title "Micro-Pico Tiny Monosynth")
-    (date "2022-08-28")
-    (rev "0.1")
+    (date "2022-10-06")
+    (rev "1.0")
     (comment 1 "creativecommons.org/licences/by/4.0")
     (comment 2 "Licence: CC by 4.0")
@@
     (stroke (width 0) (type default) (color 0 0 0 0))
   )
+  (wire (pts (xy 40.64 60.96) (xy 90.17 60.96))
+    (stroke (width 0) (type default) (color 0 0 0 0))
+  )
   (wire (pts (xy 72.39 99.06) (xy 81.28 99.06))
     (stroke (width 0) (type default) (color 0 0 0 0))
@@
   (hierarchical_label "VCA_CV" (shape output) (at 237.49 137.16 0)
     (effects (font (size 1.27 1.27)) (justify left))
+  )
+  (hierarchical_label "LFO_DEPTH_CV" (shape input) (at 40.64 60.96 180)
+    (effects (font (size 1.27 1.27)) (justify right))
   )
   (hierarchical_label "GATE_IN" (shape input) (at 40.64 99.06 180)
@@
       (effects (font (size 1.27 1.27)) (justify right))
     )
-  )
+    (pin "DEPTH_CV_IN" input (at 90.17 60.96 180)
+      (effects (font (size 1.27 1.27)) (justify left))
+    )
+  )
