File: main_pcb/kicad_6/PWM_CV_scaler.kicad_sch (KiCad schematic)
At the start: 14 parts, among them J1201 aux_PWM_in, U3 TL072

Commit message: Update rev 0.1, fix VCA tails, add local 2v5 regs, change some pot footprints
Parts:
- J1201: now left out of the parts list
- R1203: value 100k -> 220k
- RV1201: value 100k -> 5k; footprint custom_footprints:Alpha_RD901F -> custom_footprints:Bourns_PTV09
Connections:
- net -2V5_REF renamed -5V_REF
Changed lines of the file:
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@@
   (title_block
     (title "Micro-Pico Tiny Monosynth")
-    (date "2022-08-18")
+    (date "2022-08-28")
     (rev "0.1")
     (comment 1 "creativecommons.org/licences/by/4.0")
@@
   (junction (at 130.81 100.33) (diameter 0) (color 0 0 0 0)
   )
-  (wire (pts (xy 69.85 92.71) (xy 73.66 92.71))
-    (stroke (width 0) (type default) (color 0 0 0 0))
-  )
   (wire (pts (xy 151.13 78.74) (xy 144.78 78.74))
     (stroke (width 0) (type default) (color 0 0 0 0))
@@
     (stroke (width 0) (type default) (color 0 0 0 0))
   )
-  (wire (pts (xy 73.66 92.71) (xy 73.66 96.52))
+  (wire (pts (xy 73.66 86.36) (xy 73.66 96.52))
     (stroke (width 0) (type default) (color 0 0 0 0))
   )
@@
   )
   (wire (pts (xy 151.13 91.44) (xy 151.13 78.74))
+    (stroke (width 0) (type default) (color 0 0 0 0))
+  )
+  (wire (pts (xy 64.77 86.36) (xy 73.66 86.36))
     (stroke (width 0) (type default) (color 0 0 0 0))
   )
@@
     (effects (font (size 1.27 1.27)) (justify left bottom))
   )
-  (global_label "-2V5_REF" (shape input) (at 69.85 92.71 180) (fields_autoplaced)
+  (global_label "-5V_REF" (shape input) (at 64.77 86.36 180) (fields_autoplaced)
     (effects (font (size 1.27 1.27)) (justify right))
-    (property "Intersheet References" "${INTERSHEET_REFS}" (id 0) (at 57.8817 92.7894 0)
+    (property "Intersheet References" "${INTERSHEET_REFS}" (id 0) (at 54.0112 86.4394 0)
       (effects (font (size 1.27 1.27)) (justify right) hide)
     )
@@
       (effects (font (size 1.27 1.27)) (justify right))
     )
-    (property "Value" "100k" (id 1) (at 71.12 101.5999 0)
-      (effects (font (size 1.27 1.27)) (justify right))
-    )
-    (property "Footprint" "custom_footprints:Alpha_RD901F" (id 2) (at 73.66 100.33 0)
+    (property "Value" "5k" (id 1) (at 71.12 101.5999 0)
+      (effects (font (size 1.27 1.27)) (justify right))
+    )
+    (property "Footprint" "custom_footprints:Bourns_PTV09" (id 2) (at 73.66 100.33 0)
       (effects (font (size 1.27 1.27)) hide)
     )
@@
     (in_bom yes) (on_board yes)
     (property "Reference" "R1203" (id 0) (at 113.03 95.25 90))
-    (property "Value" "100k" (id 1) (at 113.03 97.79 90))
+    (property "Value" "220k" (id 1) (at 113.03 97.79 90))
     (property "Footprint" "Resistor_SMD:R_0603_1608Metric" (id 2) (at 113.03 102.108 90)
       (effects (font (size 1.27 1.27)) hide)
@@
   )
   (symbol (lib_id "Connector_Generic:Conn_01x01") (at 90.17 69.85 0) (mirror y) (unit 1)
-    (in_bom yes) (on_board yes) (fields_autoplaced)
+    (in_bom no) (on_board yes) (fields_autoplaced)
     (property "Reference" "J1201" (id 0) (at 90.17 63.5 0))
     (property "Value" "aux_PWM_in" (id 1) (at 90.17 66.04 0))
